File: battery-sensor.kicad_sch (KiCad schematic)
At the start: 22 parts, among them J1 Conn_01x06_Pin, J10 Conn_01x03_Pin, J2 Conn_01x06_Pin, J3 Conn_01x06_Pin, J4 Conn_01x08_Pin, J5 Conn_01x06_Pin, J6 Conn_01x02_Pin, J7 Conn_01x02_Pin, J8 Conn_01x02_Pin, J9 Conn_01x02_Pin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

Commit message: Increase mounting hole size to account for small size variations of the plastic enclosures.
Parts:
- H1, H2, H3, H4: footprint MountingHole:MountingHole_2.7mm_M2.5_ISO7380 -> MountingHole:MountingHole_3.5mm
Changed lines of the file:
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@@
 			)
 		)
-		(property "Footprint" "MountingHole:MountingHole_2.7mm_M2.5_ISO7380"
+		(property "Footprint" "MountingHole:MountingHole_3.5mm"
 			(at 151.13 181.61 0)
 			(hide yes)
@@
 			)
 		)
-		(property "Footprint" "MountingHole:MountingHole_2.7mm_M2.5_ISO7380"
+		(property "Footprint" "MountingHole:MountingHole_3.5mm"
 			(at 151.13 175.26 0)
 			(hide yes)
@@
 			)
 		)
-		(property "Footprint" "MountingHole:MountingHole_2.7mm_M2.5_ISO7380"
+		(property "Footprint" "MountingHole:MountingHole_3.5mm"
 			(at 151.13 187.96 0)
 			(hide yes)
@@
 			)
 		)
-		(property "Footprint" "MountingHole:MountingHole_2.7mm_M2.5_ISO7380"
+		(property "Footprint" "MountingHole:MountingHole_3.5mm"
 			(at 151.13 168.91 0)
 			(hide yes)
